Commit message: Added eros urdf model with inertia

File: src/nimbro/hardware/nimbro_op_model/robots/eros_base.xacro (robot description, xacro)
@@ -5,22 +5,37 @@
       <color rgba="0.1 0.1 0.1 1" />
     </material>
+    <material name="white">
+      <color rgba="0.8 0.8 0.8 1" />
+    </material>
+<!-- ======================================================
+ Name        : eros.urdf / Eros Robot Model
+ Author      : rokhmat@eros
+ Version     : 1.0
+ Copyright   : EROS <erojaya.bejo> Team
+ Description :
+======================================================
+ -->
     <link name="trunk_link">
       <inertial>
-        <origin xyz="-0.016856 -0.00019822 0.019225" rpy="0 0 0" />
-        <mass value="1.8051" />
-        <inertia ixx="0.016444" ixy="1.4574E-05" ixz="0.00048254"
-        iyy="0.013972" iyz="5.0355E-06" izz="0.0064508" />
-      </inertial>
-      <visual>
-        <origin xyz="0 0 0.01" rpy="0 0 0" />
-        <geometry>
-          <box size="0.12 0.125 0.185" />
-        </geometry>
-        <material name="black" />
-      </visual>
-      <collision>
-        <origin xyz="0 0 0.01" rpy="0 0 0" />
-        <geometry>
-          <box size="0.12 0.125 0.185" />
+        <origin xyz="-0.012677 -6.4526E-05 -0.024311" rpy="0 0 0" />
+        <mass value="2.045" />
+        <inertia ixx="0.00804781" ixy="-0.00001059" ixz="-0.00013634"
+        iyy="0.00727409" iyz="-0.00000696" izz="0.00540421" />
+      </inertial>
+      <visual>
+        <origin xyz="0 0 0" rpy="0 0 0" />
+        <geometry>
+          <!-- <box size="0.12 0.125 0.185" /> -->
+          <mesh
+          filename="package://nimbro_op_model/mesh/eros/trunk_link.STL" />
+        </geometry>
+        <material name="white" />
+      </visual>
+      <collision>
+        <origin xyz="0 0 0" rpy="0 0 0" />
+        <geometry>
+          <!-- <box size="0.12 0.125 0.185" /> -->
+          <mesh
+          filename="package://nimbro_op_model/mesh/eros/trunk_link.STL" />
         </geometry>
       </collision>
@@ -28,25 +43,29 @@
     <link name="right_hip_yaw_link">
       <inertial>
-        <origin xyz="4.7878E-16 2.8449E-16 -0.013803" rpy="0 0 0" />
-        <mass value="0.073374" />
-        <inertia ixx="2.6774E-05" ixy="1.5536E-19" ixz="-9.0622E-19"
-        iyy="0.00011478" iyz="-2.2736E-19" izz="0.00010743" />
-      </inertial>
-      <visual>
-        <origin xyz="0 0 0" rpy="0 0 0" />
-        <geometry>
-          <box size="0.06 0.05 0.03" />
-        </geometry>
-        <material name="black" />
-      </visual>
-      <collision>
-        <origin xyz="0 0 0" rpy="0 0 0" />
-        <geometry>
-          <box size="0.06 0.05 0.03" />
+        <origin xyz="0.0032766 -0.0013724 -0.0095963" rpy="0 0 0" />
+        <mass value="0.025" />
+        <inertia ixx="0.00000507" ixy="0.00000000" ixz="0.00000012"
+        iyy="0.00001647" iyz="-0.00000021" izz="0.00001529" />
+      </inertial>
+      <visual>
+        <origin xyz="0 0 0" rpy="0 0 0" />
+        <geometry>
+          <!-- <box size="0.06 0.05 0.03" /> -->
+          <mesh
+          filename="package://nimbro_op_model/mesh/eros/right_hip_yaw_link.STL" />
+        </geometry>
+        <material name="black" />
+      </visual>
+      <collision>
+        <origin xyz="0 0 0" rpy="0 0 0" />
+        <geometry>
+          <!-- <box size="0.06 0.05 0.03" /> -->
+          <mesh
+          filename="package://nimbro_op_model/mesh/eros/right_hip_yaw_link.STL" />
         </geometry>
       </collision>
     </link>
     <joint name="right_hip_yaw" type="continuous">
-      <origin xyz="0 -0.055 -0.0936" rpy="0 0 0" />
+      <origin xyz="0 -0.04773 -0.08789" rpy="0 0 0" />
       <parent link="trunk_link" />
       <child link="right_hip_yaw_link" />
@@ -55,52 +74,60 @@
     <link name="right_hip_roll_link">
       <inertial>
-        <origin xyz="0.010896 0.00023756 -0.014538" rpy="0 0 0" />
-        <mass value="0.35903" />
-        <inertia ixx="0.00015503" ixy="1.738E-06" ixz="8.5148E-06"
-        iyy="0.0003299" iyz="2.4403E-07" izz="0.0002782" />
-      </inertial>
-      <visual>
-        <origin xyz="0 0 0" rpy="0 0 0" />
-        <geometry>
-          <box size="0.1 0.05 0.05" />
-        </geometry>
-        <material name="black" />
-      </visual>
-      <collision>
-        <origin xyz="0 0 0" rpy="0 0 0" />
-        <geometry>
-          <box size="0.1 0.05 0.05" />
+        <origin xyz="-0.0191155528309945 -1.96042503744776E-05 -0.0140757799459858" rpy="0 0 0" />
+        <mass value="0.31" />
+        <inertia ixx="0.00011858" ixy="-0.00000010" ixz="0.00002045"
+        iyy="0.00034098" iyz="-0.00000080" izz="0.00029886" />
+      </inertial>
+      <visual>
+        <origin xyz="0 0 0" rpy="0 0 0" />
+        <geometry>
+          <!-- <box size="0.1 0.05 0.05" /> -->
+          <mesh
+          filename="package://nimbro_op_model/mesh/eros/right_hip_roll_link.STL" />
+        </geometry>
+        <material name="white" />
+      </visual>
+      <collision>
+        <origin xyz="0 0 0" rpy="0 0 0" />
+        <geometry>
+          <!-- <box size="0.1 0.05 0.05" /> -->
+          <mesh
+          filename="package://nimbro_op_model/mesh/eros/right_hip_roll_link.STL" />
         </geometry>
       </collision>
     </link>
     <joint name="right_hip_roll" type="continuous">
-      <origin xyz="-0.00721428464376577 0 -0.0338" rpy="0 0 0" />
+      <origin xyz="4.26083784947351E-05 0 -0.038" rpy="0 0 0" />
       <parent link="right_hip_yaw_link" />
       <child link="right_hip_roll_link" />
-      <axis xyz="1 0 0" />
+      <axis xyz="-1 0 0" />
     </joint>
     <link name="right_thigh_link">
       <inertial>
-        <origin xyz="0.0038549 0.00023828 -0.1495" rpy="0 0 0" />
-        <mass value="0.38276" />
-        <inertia ixx="0.0020951" ixy="1.8755E-07" ixz="-0.00017816"
-        iyy="0.0020043" iyz="-5.4867E-06" izz="0.00027919" />
-      </inertial>
-      <visual>
-        <origin xyz="0 0 -0.03" rpy="0 0 0" />
-        <geometry>
-          <box size="0.05 0.05 0.12" />
-        </geometry>
-        <material name="black" />
-      </visual>
-      <collision>
-        <origin xyz="0 0 -0.03" rpy="0 0 0" />
-        <geometry>
-          <box size="0.05 0.05 0.12" />
+        <origin xyz="0.0054277 0.00034049 -0.082269" rpy="0 0 0" />
+        <mass value="0.19" />
+        <inertia ixx="0.00019524" ixy="-0.00000037" ixz="0.00001202"
+        iyy="0.00017893" iyz="-0.00000009" izz="0.00008079" />
+      </inertial>
+      <visual>
+        <origin xyz="0 0 0" rpy="0 0 0" />
+        <geometry>
+          <!-- <box size="0.05 0.05 0.12" /> -->
+          <mesh
+          filename="package://nimbro_op_model/mesh/eros/right_thigh_link.STL" />
+        </geometry>
+        <material name="black" />
+      </visual>
+      <collision>
+        <origin xyz="0 0 0" rpy="0 0 0" />
+        <geometry>
+          <!-- <box size="0.05 0.05 0.12" /> -->
+          <mesh
+          filename="package://nimbro_op_model/mesh/eros/right_thigh_link.STL" />
         </geometry>
       </collision>
     </link>
     <joint name="right_hip_pitch" type="continuous">
-      <origin xyz="0.0151571423218829 0 -0.03" rpy="0 0 0" />
+      <origin xyz="0 0.000272865563695893 0" rpy="0 0 0" />
       <parent link="right_hip_roll_link" />
       <child link="right_thigh_link" />
@@ -109,25 +136,29 @@
     <link name="right_shank_link">
       <inertial>
-        <origin xyz="-0.0033779 6.578E-10 -0.10469" rpy="0 0 0" />
-        <mass value="0.20549" />
-        <inertia ixx="0.0011378" ixy="-2.8771E-12" ixz="9.7123E-05"
-        iyy="0.0010393" iyz="-1.4479E-11" izz="0.00019656" />
-      </inertial>
-      <visual>
-        <origin xyz="0 0 -0.03" rpy="0 0 0" />
-        <geometry>
-          <box size="0.05 0.05 0.12" />
-        </geometry>
-        <material name="black" />
-      </visual>
-      <collision>
-        <origin xyz="0 0 -0.03" rpy="0 0 0" />
-        <geometry>
-          <box size="0.05 0.05 0.12" />
+        <origin xyz="0.0084982 1.6653E-16 -0.052577" rpy="0 0 0" />
+        <mass value="0.045" />
+        <inertia ixx="0.00006993" ixy="0.00000000" ixz="0.00000302"
+        iyy="0.00005366" iyz="0.00000000" izz="0.00002875" />
+      </inertial>
+      <visual>
+        <origin xyz="0 0 0" rpy="0 0 0" />
+        <geometry>
+          <!-- <box size="0.05 0.05 0.12" /> -->
+          <mesh
+          filename="package://nimbro_op_model/mesh/eros/right_shank_link.STL" />
+        </geometry>
+        <material name="black" />
+      </visual>
+      <collision>
+        <origin xyz="0 0 0" rpy="0 0 0" />
+        <geometry>
+          <!-- <box size="0.05 0.05 0.12" /> -->
+          <mesh
+          filename="package://nimbro_op_model/mesh/eros/right_shank_link.STL" />
         </geometry>
       </collision>
     </link>
     <joint name="right_knee_pitch" type="continuous">
-      <origin xyz="0 0 -0.1" rpy="0 0 0" />
+      <origin xyz="0.000139526375362783 0.000754789894666347 -0.110000000000033" rpy="0 0 0" />
       <parent link="right_thigh_link" />
       <child link="right_shank_link" />
@@ -136,25 +167,29 @@
     <link name="right_ankle_link">
       <inertial>
-        <origin xyz="-0.019434 0.00024988 0.014536" rpy="0 0 0" />
-        <mass value="0.35844" />
-        <inertia ixx="0.00015501" ixy="1.7299E-06" ixz="-8.5156E-06"
-        iyy="0.00032958" iyz="-2.4435E-07" izz="0.00027786" />
-      </inertial>
-      <visual>
-        <origin xyz="0 0 0" rpy="0 0 0" />
-        <geometry>
-          <box size="0.09 0.05 0.05" />
-        </geometry>
-        <material name="black" />
-      </visual>
-      <collision>
-        <origin xyz="0 0 0" rpy="0 0 0" />
-        <geometry>
-          <box size="0.09 0.05 0.05" />
+        <origin xyz="-0.019428 -1.1817E-05 0.013886" rpy="0 0 0" />
+        <mass value="0.315" />
+        <inertia ixx="0.00011956" ixy="-0.00000016" ixz="-0.00002101"
+        iyy="0.00035616" iyz="0.00000088" izz="0.00031274" />
+      </inertial>
+      <visual>
+        <origin xyz="0 0 0" rpy="0 0 0" />
+        <geometry>
+          <!-- <box size="0.09 0.05 0.05" /> -->
+          <mesh
+          filename="package://nimbro_op_model/mesh/eros/right_ankle_link.STL" />
+        </geometry>
+        <material name="white" />
+      </visual>
+      <collision>
+        <origin xyz="0 0 0" rpy="0 0 0" />
+        <geometry>
+          <!-- <box size="0.09 0.05 0.05" /> -->
+          <mesh
+          filename="package://nimbro_op_model/mesh/eros/right_ankle_link.STL" />
         </geometry>
       </collision>
     </link>
     <joint name="right_ankle_pitch" type="continuous">
-      <origin xyz="0 0 -0.1" rpy="0 0 0" />
+      <origin xyz="0 -0.000151355466657691 -0.115" rpy="0 0 0" />
       <parent link="right_shank_link" />
       <child link="right_ankle_link" />
@@ -163,28 +198,32 @@
     <link name="right_foot_link">
       <inertial>
-        <origin xyz="0.003669 -0.0081165 -0.030903" rpy="0 0 0" />
-        <mass value="0.1488" />
-        <inertia ixx="0.00018527" ixy="-1.1504E-05" ixz="-7.2667E-06"
-        iyy="0.00060485" iyz="5.8883E-06" izz="0.00075217" />
-      </inertial>
-      <visual>
-        <origin xyz="0 0 -0.01" rpy="0 0 0" />
-        <geometry>
-          <box size="0.125 0.08 0.03" />
-        </geometry>
-        <material name="black" />
-      </visual>
-      <collision>
-        <origin xyz="0 0 -0.01" rpy="0 0 0" />
-        <geometry>
-          <box size="0.125 0.08 0.03" />
+        <origin xyz="0.0032874 -0.0054641 -0.034665" rpy="0 0 0" />
+        <mass value="0.08" />
+        <inertia ixx="0.00006014" ixy="-0.00000011" ixz="-0.00000006"
+        iyy="0.00013602" iyz="0.00000082" izz="0.00018868" />
+      </inertial>
+      <visual>
+        <origin xyz="0 0 0" rpy="0 0 0" />
+        <geometry>
+          <!-- <box size="0.125 0.08 0.03" /> -->
+          <mesh
+          filename="package://nimbro_op_model/mesh/eros/right_foot_link.STL" />
+        </geometry>
+        <material name="black" />
+      </visual>
+      <collision>
+        <origin xyz="0 0 0" rpy="0 0 0" />
+        <geometry>
+          <!-- <box size="0.125 0.08 0.03" /> -->
+          <mesh
+          filename="package://nimbro_op_model/mesh/eros/right_foot_link.STL" />
         </geometry>
       </collision>
     </link>
     <joint name="right_ankle_roll" type="continuous">
-      <origin xyz="0 0 0" rpy="0 0 0" />
+      <origin xyz="-5.05476446036046E-05 0 0" rpy="0 0 0" />
       <parent link="right_ankle_link" />
       <child link="right_foot_link" />
-      <axis xyz="1 0 0" />
+      <axis xyz="-1 0 0" />
     </joint>
     <link name="right_foot_plane_link">
@@ -198,25 +237,29 @@
     <link name="left_hip_yaw_link">
       <inertial>
-        <origin xyz="4.996E-16 2.5674E-16 -0.013803" rpy="0 0 0" />
-        <mass value="0.073374" />
-        <inertia ixx="2.6774E-05" ixy="1.9727E-19" ixz="-8.7961E-19"
-        iyy="0.00011478" iyz="-2.3128E-19" izz="0.00010743" />
-      </inertial>
-      <visual>
-        <origin xyz="0 0 0" rpy="0 0 0" />
-        <geometry>
-          <box size="0.06 0.05 0.03" />
-        </geometry>
-        <material name="black" />
-      </visual>
-      <collision>
-        <origin xyz="0 0 0" rpy="0 0 0" />
-        <geometry>
-          <box size="0.06 0.05 0.03" />
+        <origin xyz="0.0032766 0.0013724 -0.0095963" rpy="0 0 0" />
+        <mass value="0.025" />
+        <inertia ixx="0.00000507" ixy="0.00000000" ixz="0.00000012"
+        iyy="0.00001647" iyz="0.00000021" izz="0.00001529" />
+      </inertial>
+      <visual>
+        <origin xyz="0 0 0" rpy="0 0 0" />
+        <geometry>
+          <!-- <box size="0.06 0.05 0.03" /> -->
+          <mesh
+          filename="package://nimbro_op_model/mesh/eros/left_hip_yaw_link.STL" />
+        </geometry>
+        <material name="black" />
+      </visual>
+      <collision>
+        <origin xyz="0 0 0" rpy="0 0 0" />
+        <geometry>
+          <!-- <box size="0.06 0.05 0.03" /> -->
+          <mesh
+          filename="package://nimbro_op_model/mesh/eros/left_hip_yaw_link.STL" />
         </geometry>
       </collision>
     </link>
     <joint name="left_hip_yaw" type="continuous">
-      <origin xyz="0 0.055 -0.0936" rpy="0 0 0" />
+      <origin xyz="0 0.04773 -0.08789" rpy="0 0 0" />
       <parent link="trunk_link" />
       <child link="left_hip_yaw_link" />
@@ -225,54 +268,62 @@
 <link name="left_hip_roll_link">
       <inertial>
-        <origin xyz="-0.019434 -0.0002499 -0.014536" rpy="0 0 0" />
-        <mass value="0.35844" />
+        <origin xyz="-0.019116 2.1864E-05 -0.014076" rpy="0 0 0" />
+        <mass value="0.31" />
         <!-- TODO: the origin was shifted by -0.0012 and this was not updated -->
-        <inertia ixx="0.00015501" ixy="-1.7299E-06" ixz="8.5156E-06"
-        iyy="0.00032958" iyz="-2.4435E-07" izz="0.00027786" />
-      </inertial>
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