Commit message: Added generated urdf robot model

File: src/nimbro/hardware/nimbro_op_model/robots/urdf/eros.urdf (robot description, URDF)
Before this commit: robot eros, 40 links, 39 joints
Links:
- removed link base_link
- removed link kepala
- removed link leher
- removed link lengan_bawah_kanan
- removed link lengan_bawah_kiri
- removed link link_betis_kanan
- removed link link_betis_kiri
- removed link link_paha_kanan
- removed link link_paha_kiri
- removed link link_servo_bahu_kanan
- removed link link_servo_bahu_kiri
- removed link link_siku_kanan
- removed link link_siku_kiri
- removed link servo_bahu_pitch_kanan
- removed link servo_bahu_pitch_kiri
- removed link servo_bahu_roll_kanan
- removed link servo_bahu_roll_kiri
- removed link servo_engkle_pitch_kanan
- removed link servo_engkle_pitch_kiri
- removed link servo_engkle_roll_kanan
- removed link servo_engkle_roll_kiri
- removed link servo_hip_pitch_kanan
- removed link servo_hip_pitch_kiri
- removed link servo_hip_roll_kanan
- removed link servo_hip_roll_kiri
- removed link servo_hip_yaw_kanan
- removed link servo_hip_yaw_kiri
- removed link servo_leher_y
- removed link servo_lutut_kanan
- removed link servo_lutut_kiri
- removed link servo_siku_pitch_kanan
- removed link servo_siku_pitch_kiri
- removed link telapak_kaki_kanan
- removed link telapak_kaki_kanan_eof
- removed link telapak_kaki_kiri
- removed link telapak_kaki_kiri_eof
- removed link ujung_tangan_kanan
- removed link ujung_tangan_kiri
- added link head_link, mass 0.11; collision mesh filename=package://nimbro_op_model/mesh/eros/head_link.STL; visual mesh filename=package://nimbro_op_model/mesh/eros/head_link.STL
- added link left_ankle_link, mass 0.315; collision mesh filename=package://nimbro_op_model/mesh/eros/left_ankle_link.STL; visual mesh filename=package://nimbro_op_model/mesh/eros/left_ankle_link.STL
- added link left_foot_link, mass 0.08; collision mesh filename=package://nimbro_op_model/mesh/eros/left_foot_link.STL; visual mesh filename=package://nimbro_op_model/mesh/eros/left_foot_link.STL
- added link left_foot_plane_link
- added link left_hip_roll_link, mass 0.31; collision mesh filename=package://nimbro_op_model/mesh/eros/left_hip_roll_link.STL; visual mesh filename=package://nimbro_op_model/mesh/eros/left_hip_roll_link.STL
- added link left_hip_yaw_link, mass 0.025; collision mesh filename=package://nimbro_op_model/mesh/eros/left_hip_yaw_link.STL; visual mesh filename=package://nimbro_op_model/mesh/eros/left_hip_yaw_link.STL
- added link left_lower_arm_link, mass 0.065; collision mesh filename=package://nimbro_op_model/mesh/eros/left_lower_arm_link.STL; visual mesh filename=package://nimbro_op_model/mesh/eros/left_lower_arm_link.STL
- added link left_shank_link, mass 0.045; collision mesh filename=package://nimbro_op_model/mesh/eros/left_shank_link.STL; visual mesh filename=package://nimbro_op_model/mesh/eros/left_shank_link.STL
- added link left_shoulder_pitch_link, mass 0.015; collision mesh filename=package://nimbro_op_model/mesh/eros/left_shoulder_pitch_lin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; visual mesh filename=package://nimbro_op_model/mesh/eros/left_shoulder_pitch_lin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
- added link left_thigh_link, mass 0.19; collision mesh filename=package://nimbro_op_model/mesh/eros/left_thigh_link.STL; visual mesh filename=package://nimbro_op_model/mesh/eros/left_thigh_link.STL
- added link left_upper_arm_link, mass 0.19; collision mesh filename=package://nimbro_op_model/mesh/eros/left_upper_arm_link.STL; visual mesh filename=package://nimbro_op_model/mesh/eros/left_upper_arm_link.STL
- added link neck_link, mass 0.095; collision mesh filename=package://nimbro_op_model/mesh/eros/neck_link.STL; visual mesh filename=package://nimbro_op_model/mesh/eros/neck_link.STL
- added link right_ankle_link, mass 0.315; collision mesh filename=package://nimbro_op_model/mesh/eros/right_ankle_link.STL; visual mesh filename=package://nimbro_op_model/mesh/eros/right_ankle_link.STL
- added link right_foot_link, mass 0.08; collision mesh filename=package://nimbro_op_model/mesh/eros/right_foot_link.STL; visual mesh filename=package://nimbro_op_model/mesh/eros/right_foot_link.STL
- added link right_foot_plane_link
- added link right_hip_roll_link, mass 0.31; collision mesh filename=package://nimbro_op_model/mesh/eros/right_hip_roll_link.STL; visual mesh filename=package://nimbro_op_model/mesh/eros/right_hip_roll_link.STL
- added link right_hip_yaw_link, mass 0.025; collision mesh filename=package://nimbro_op_model/mesh/eros/right_hip_yaw_link.STL; visual mesh filename=package://nimbro_op_model/mesh/eros/right_hip_yaw_link.STL
- added link right_lower_arm_link, mass 0.065; collision mesh filename=package://nimbro_op_model/mesh/eros/right_lower_arm_link.STL; visual mesh filename=package://nimbro_op_model/mesh/eros/right_lower_arm_link.STL
- added link right_shank_link, mass 0.045; collision mesh filename=package://nimbro_op_model/mesh/eros/right_shank_link.STL; visual mesh filename=package://nimbro_op_model/mesh/eros/right_shank_link.STL
- added link right_shoulder_pitch_link, mass 0.015; collision mesh filename=package://nimbro_op_model/mesh/eros/right_shoulder_pitch_li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; visual mesh filename=package://nimbro_op_model/mesh/eros/right_shoulder_pitch_li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
- added link right_thigh_link, mass 0.19; collision mesh filename=package://nimbro_op_model/mesh/eros/right_thigh_link.STL; visual mesh filename=package://nimbro_op_model/mesh/eros/right_thigh_link.STL
- added link right_upper_arm_link, mass 0.19; collision mesh filename=package://nimbro_op_model/mesh/eros/right_upper_arm_link.STL; visual mesh filename=package://nimbro_op_model/mesh/eros/right_upper_arm_link.STL
- link camera_optical: mass 0.126 -> 0.095; geometry collision mesh filename=package://nimbro_op_model/mesh/eros/camera_optical.STL; visual mesh filename=package://nimbro_op_model/mesh/eros/camera_optical.STL
- link trunk_link: mass 1 -> 2.045; geometry collision mesh filename=package://nimbro_op_model/mesh/eros/trunk_link.STL; visual mesh filename=package://nimbro_op_model/mesh/eros/trunk_link.STL
Joints:
- removed joint base_to_hip_kanan
- removed joint base_to_hip_kiri
- removed joint kaki_kanan_eof
- removed joint kaki_kiri_eof
- removed joint kamera_eof
- removed joint leher_to_bahu_kanan
- removed joint leher_to_bahu_kiri
- removed joint leher_to_base
- removed joint link_lengan_atas_kanan
- removed joint link_lengan_atas_kiri
- removed joint link_lengan_bawah_kanan
- removed joint link_lengan_bawah_kiri
- removed joint link_servo_engkle_kanan
- removed joint link_servo_engkle_kiri
- removed joint link_servo_lutut_kanan
- removed joint link_servo_lutut_kiri
- removed joint perut_to_base
- removed joint tangan_kanan_eof
- removed joint tangan_kiri_eof
- added joint camera_joint: type fixed, parent head_link, child camera_optical, origin xyz=0.012 0 0.045383 rpy=-1.57079632679489 0 -1.57079632679489, axis 0 0 0
- added joint left_foot_plane_joint: type fixed, parent left_foot_link, child left_foot_plane_link, origin xyz=0.0009 0.011 -0.039 rpy=0 0 0
- added joint right_foot_plane_joint: type fixed, parent right_foot_link, child right_foot_plane_link, origin xyz=0.0009 -0.011 -0.039 rpy=0 0 0
- joint head_pitch: axis 1 0 0 -> 0 1 0; child kepala -> head_link; limit lower=-1.57 upper=1.57 effort=300 velocity=0.1 -> (none); origin xyz=0 0 0.0  rpy=0 0 0 -> xyz=0.00400000000000034 0.000266141079259985 0.0222 rpy=0 0 0; parent servo_leher_y -> neck_link
- joint left_ankle_pitch: axis 1 0 0 -> 0 1 0; child servo_engkle_roll_kiri -> left_ankle_link; limit lower=-3.14 upper=3.14 effort=300 velocity=0.1 -> (none); origin xyz=0 0.0 -0.11 -> xyz=0 -0.000151355466657691 -0.115 rpy=0 0 0; parent link_betis_kiri -> left_shank_link
- joint left_ankle_roll: axis 0 1 0 -> -1 0 0; child telapak_kaki_kiri -> left_foot_link; limit lower=-3.14 upper=3.14 effort=300 velocity=0.1 -> (none); origin xyz=0 0.025 0 -> xyz=-5.05476446036046E-05 0 0          rpy=0 0 0; parent servo_engkle_pitch_kiri -> left_ankle_link
- joint left_elbow_pitch: axis 0 0 -1 -> 0 -1 0; child servo_siku_pitch_kiri -> left_lower_arm_link; origin xyz=-0.070 0 0. rpy=0 0 0 -> xyz=0.0210000000000005 -5.04771949249166E-05 -0.0934000000000005 rpy=0 0 0; parent link_siku_kiri -> left_upper_arm_link
- joint left_hip_pitch: axis -1 0 0 -> 0 1 0; child link_paha_kiri -> left_thigh_link; limit lower=-3.14 upper=3.14 effort=300 velocity=0.1 -> (none); origin xyz=0 0.0 0 -> xyz=0 0.000272865563695893 0 rpy=0 0 0; parent servo_hip_roll_kiri -> left_hip_roll_link
- joint left_hip_roll: axis 0 -1 0 -> -1 0 0; child servo_hip_roll_kiri -> left_hip_roll_link; limit lower=-3.14 upper=3.14 effort=300 velocity=0.1 -> (none); origin xyz=0 0.02 0 -> xyz=4.26083784947351E-05 0 -0.038 rpy=0 0 0; parent servo_hip_pitch_kiri -> left_hip_yaw_link
- joint left_hip_yaw: axis 0 0 -1 -> 0 0 1; child servo_hip_pitch_kiri -> left_hip_yaw_link; limit lower=-3.14 upper=3.14 effort=300 velocity=0.1 -> (none); origin xyz=0 0 -0.060 -> xyz=0 0.04773 -0.08789 rpy=0 0 0; parent servo_hip_yaw_kiri -> trunk_link
- joint left_knee_pitch: axis -1 0 0 -> 0 1 0; child link_betis_kiri -> left_shank_link; limit lower=-3.14 upper=3.14 effort=300 velocity=0.1 -> (none); origin xyz=0 0.0 -0.01 -> xyz=0.000139526375362783 0.000754789894666347 -0.110000000000033 rpy=0 0 0; parent servo_lutut_kiri -> left_thigh_link
- joint left_shoulder_pitch: axis -1 0 0 -> 0 1 0; child link_servo_bahu_kiri -> left_shoulder_pitch_link; limit lower=-3.14 upper=3.14 effort=300 velocity=0.1 -> (none); origin xyz=-0.030 0 0 rpy=0 0 0 -> xyz=0 0.0656181565488089 0.0548 rpy=0 0 0; parent servo_bahu_roll_kiri -> trunk_link
- joint left_shoulder_roll: axis 0 -1 0 -> 1 0 0; child servo_bahu_pitch_kiri -> left_upper_arm_link; limit lower=-2.0 upper=2.0 effort=300 velocity=0.1 -> (none); origin xyz=-0.010 0 -0.015 rpy=0 0 0 -> xyz=-0.00027665735414488 0.0240000000000005 -0.0159973139955498 rpy=0 0 0; parent link_servo_bahu_kiri -> left_shoulder_pitch_link
- joint neck_yaw: child servo_leher_y -> neck_link; limit lower=-3.14 upper=3.14 effort=300 velocity=0.1 -> (none); origin xyz=0 0 0.05  rpy=0 0 0 -> xyz=0 0 0.077862 rpy=0 0 0; parent leher -> trunk_link
- joint right_ankle_pitch: axis -1 0 0 -> 0 1 0; child servo_engkle_roll_kanan -> right_ankle_link; limit lower=-3.14 upper=3.14 effort=300 velocity=0.1 -> (none); origin xyz=0 0.0 -0.11 -> xyz=0 -0.000151355466657691 -0.115 rpy=0 0 0; parent link_betis_kanan -> right_shank_link
- joint right_ankle_roll: axis 0 1 0 -> -1 0 0; child telapak_kaki_kanan -> right_foot_link; limit lower=-3.14 upper=3.14 effort=300 velocity=0.1 -> (none); origin xyz=0 0.025 0 -> xyz=-5.05476446036046E-05 0 0 rpy=0 0 0; parent servo_engkle_pitch_kanan -> right_ankle_link
- joint right_elbow_pitch: axis 0 0 -1 -> 0 -1 0; child servo_siku_pitch_kanan -> right_lower_arm_link; limit lower=-1.57 upper=1.57 effort=300 velocity=0.1 -> (none); origin xyz=0.070 0 0. rpy=0 0 0 -> xyz=0.0210000000000005 -5.04771949249166E-05 -0.0934000000000005 rpy=0 0 0; parent link_siku_kanan -> right_upper_arm_link
- joint right_hip_pitch: axis 1 0 0 -> 0 1 0; child link_paha_kanan -> right_thigh_link; limit lower=-3.14 upper=3.14 effort=300 velocity=0.1 -> (none); origin xyz=0 0.0 0 -> xyz=0 0.000272865563695893 0 rpy=0 0 0; parent servo_hip_roll_kanan -> right_hip_roll_link
- joint right_hip_roll: axis 0 -1 0 -> -1 0 0; child servo_hip_roll_kanan -> right_hip_roll_link; limit lower=-3.14 upper=3.14 effort=300 velocity=0.1 -> (none); origin xyz=0 0.02 0 -> xyz=4.26083784947351E-05 0 -0.038 rpy=0 0 0; parent servo_hip_pitch_kanan -> right_hip_yaw_link
- joint right_hip_yaw: axis 0 0 -1 -> 0 0 1; child servo_hip_pitch_kanan -> right_hip_yaw_link; limit lower=-3.14 upper=3.14 effort=300 velocity=0.1 -> (none); origin xyz=0 0 -0.060 -> xyz=0 -0.04773 -0.08789 rpy=0 0 0; parent servo_hip_yaw_kanan -> trunk_link
- joint right_knee_pitch: axis 1 0 0 -> 0 1 0; child link_betis_kanan -> right_shank_link; limit lower=-3.14 upper=3.14 effort=300 velocity=0.1 -> (none); origin xyz=0 0.0 -0.01 -> xyz=0.000139526375362783 0.000754789894666347 -0.110000000000033 rpy=0 0 0; parent servo_lutut_kanan -> right_thigh_link
- joint right_shoulder_pitch: axis 1 0 0 -> 0 1 0; child link_servo_bahu_kanan -> right_shoulder_pitch_link; limit lower=-3.14 upper=3.14 effort=300 velocity=0.1 -> (none); origin xyz=0.030 0 0 rpy=0 0 0 -> xyz=0 -0.0656181565488089 0.0548 rpy=0 0 0; parent servo_bahu_roll_kanan -> trunk_link
- joint right_shoulder_roll: axis 0 -1 0 -> 1 0 0; child servo_bahu_pitch_kanan -> right_upper_arm_link; limit lower=-2 upper=2 effort=300 velocity=0.1 -> (none); origin xyz=0.010 0 -0.015 rpy=0 0 0 -> xyz=-0.00027665735414488 -0.0240000000000005 -0.0159973139955498 rpy=0 0 0; parent link_servo_bahu_kanan -> right_shoulder_pitch_link
